File: software/geiger/wiring_diagram.sch (EAGLE design)
At the start: 0 parts

Commit message: the diagram when using one of my attiny breakouts (stuff on the board [like ISP header, bypass cap etc] not pictured, also the footprint is slightly wider)
Parts:
- added 5VREG: 7505, dp_devices:IC_VREG_3PINS-TO-220
- added BAT, SPEAKER: (no value), pinhead:PINHD-1X2
- added MEASURE, METER: (no value), pinhead:PINHD-1X3
- added SPKDRV: IRF740, transistor-power:IRF740
- added U$1: ATTINY45DIP8, SparkFun-DigitalIC:ATTINY45DIP8
Connections:
- new net 5V: 5VREG.VOUT, MEASURE.2, METER.2, U$1.VCC
- new net GND: 5VREG.GND, BAT.2, MEASURE.1, METER.1, SPKDRV.S, U$1.GND
- new net N$1: MEASURE.3, U$1.PB4(ADC2)
- new net N$2: METER.3, U$1.PB0(MOSI)
- new net N$3: SPEAKER.1, SPKDRV.D
- new net N$5: SPKDRV.G, U$1.PB1(MISO)
- new net V+: 5VREG.VIN, BAT.1, SPEAKER.2
